File: 26-313xA/coco2/peripherals.sch (KiCad schematic (older format))
At the start: 47 parts, among them CN2 Conn_01x16_Female, IC4 6821, IC5 SC67331P, IC6 SC77526, IC7 SC77527P, J6 SolderJumper_2_Open, J7 Conn_01x08, Q1 KSD880O

Commit message: -updated some component part numbers. -added a bill of materials
Parts:
- D5, D6: Manufacturer part# D-GE-GEN PURP 75V -> 1N4148; Vendor part# 2368-NTE109-ND -> 1N4148FS-ND
Changed lines of the file:
@@
 F 1 "1KF20-04" V 12550 1250 50  0001 R CNN
 F 2 "Diode_THT:D_A-405_P10.16mm_Horizontal" V 12550 1300 50  0001 C CNN
-F 3 "https://www.nteinc.com/specs/100to199/pdf/nte109.pdf" V 12550 1300 50  0001 C CNN
+F 3 "https://www.onsemi.com/pdf/datasheet/1n914-d.pdf" V 12550 1300 50  0001 C CNN
 F 4 "digikey" H 12550 1300 50  0001 C CNN "Vendor"
-F 5 "2368-NTE109-ND" H 12550 1300 50  0001 C CNN "Vendor part#"
-F 6 "D-GE-GEN PURP 75V" H 12550 1300 50  0001 C CNN "Manufacturer part#"
+F 5 "1N4148FS-ND" H 12550 1300 50  0001 C CNN "Vendor part#"
+F 6 "1N4148" H 12550 1300 50  0001 C CNN "Manufacturer part#"
 	1    12550 1300
 	0    -1   -1   0
@@
 F 1 "1KF20-04" V 12550 2750 50  0001 R CNN
 F 2 "Diode_THT:D_A-405_P10.16mm_Horizontal" V 12550 2800 50  0001 C CNN
-F 3 "https://www.nteinc.com/specs/100to199/pdf/nte109.pdf" V 12550 2800 50  0001 C CNN
+F 3 "https://www.onsemi.com/pdf/datasheet/1n914-d.pdf" V 12550 2800 50  0001 C CNN
 F 4 "digikey" H 12550 2800 50  0001 C CNN "Vendor"
-F 5 "2368-NTE109-ND" H 12550 2800 50  0001 C CNN "Vendor part#"
-F 6 "D-GE-GEN PURP 75V" H 12550 2800 50  0001 C CNN "Manufacturer part#"
+F 5 "1N4148FS-ND" H 12550 2800 50  0001 C CNN "Vendor part#"
+F 6 "1N4148" H 12550 2800 50  0001 C CNN "Manufacturer part#"
 	1    12550 2800
 	0    -1   -1   0

Commit message: -Corrected some part numbers in the BOM -Updated paret numbers for some parts in the schematic.
Parts:
- C18, C2, C35, C44: Manufacturer part# FG28C0G1H103JNT06 -> RDER71H104K0K1H03B; Vendor part# 445-173474-1-ND -> 490-8814-ND
Changed lines of the file:
@@
 F 1 ".1uF" H 9050 2550 50  0000 C CNN
 F 2 "Capacitor_THT:C_Disc_D4.7mm_W2.5mm_P5.00mm" H 9250 2550 50  0001 C CNN
-F 3 " https://product.tdk.com/info/en/catalog/datasheets/leadmlcc_halogenfree_fg_en.pdf?ref_disty=digikey" H 9250 2550 50  0001 C CNN
+F 3 " https://search.murata.co.jp/Ceramy/image/img/A01X/G101/ENG/RDE_X7R_250V-1kV_E.pdf" H 9250 2550 50  0001 C CNN
 F 4 "digikey" V 9250 2550 50  0001 C CNN "Vendor"
-F 5 "445-173474-1-ND" V 9250 2550 50  0001 C CNN "Vendor part#"
-F 6 "FG28C0G1H103JNT06" V 9250 2550 50  0001 C CNN "Manufacturer part#"
+F 5 "490-8814-ND" V 9250 2550 50  0001 C CNN "Vendor part#"
+F 6 "RDER71H104K0K1H03B" V 9250 2550 50  0001 C CNN "Manufacturer part#"
 	1    9250 2550
 	-1   0    0    1
@@
 F 1 ".1uF" V 2550 4400 50  0000 C CNN
 F 2 "Capacitor_THT:C_Disc_D4.7mm_W2.5mm_P5.00mm" H 2650 4400 50  0001 C CNN
-F 3 " https://product.tdk.com/info/en/catalog/datasheets/leadmlcc_halogenfree_fg_en.pdf?ref_disty=digikey" H 2650 4400 50  0001 C CNN
+F 3 " https://search.murata.co.jp/Ceramy/image/img/A01X/G101/ENG/RDE_X7R_250V-1kV_E.pdf" H 2650 4400 50  0001 C CNN
 F 4 "digikey" V 2650 4400 50  0001 C CNN "Vendor"
-F 5 "445-173474-1-ND" V 2650 4400 50  0001 C CNN "Vendor part#"
-F 6 "FG28C0G1H103JNT06" V 2650 4400 50  0001 C CNN "Manufacturer part#"
+F 5 "490-8814-ND" V 2650 4400 50  0001 C CNN "Vendor part#"
+F 6 "RDER71H104K0K1H03B" V 2650 4400 50  0001 C CNN "Manufacturer part#"
 	1    2650 4400
 	0    -1   -1   0
@@
 F 1 ".1uF" V 2500 850 50  0000 C CNN
 F 2 "Capacitor_THT:C_Disc_D4.7mm_W2.5mm_P5.00mm" H 2600 850 50  0001 C CNN
-F 3 " https://product.tdk.com/info/en/catalog/datasheets/leadmlcc_halogenfree_fg_en.pdf?ref_disty=digikey" H 2600 850 50  0001 C CNN
+F 3 " https://search.murata.co.jp/Ceramy/image/img/A01X/G101/ENG/RDE_X7R_250V-1kV_E.pdf" H 2600 850 50  0001 C CNN
 F 4 "digikey" V 2600 850 50  0001 C CNN "Vendor"
-F 5 "445-173474-1-ND" V 2600 850 50  0001 C CNN "Vendor part#"
-F 6 "FG28C0G1H103JNT06" V 2600 850 50  0001 C CNN "Manufacturer part#"
+F 5 "490-8814-ND" V 2600 850 50  0001 C CNN "Vendor part#"
+F 6 "RDER71H104K0K1H03B" V 2600 850 50  0001 C CNN "Manufacturer part#"
 	1    2600 850
 	0    -1   -1   0
@@
 F 1 ".1uF" H 5700 4550 50  0000 C CNN
 F 2 "Capacitor_THT:C_Disc_D4.7mm_W2.5mm_P5.00mm" H 5550 4450 50  0001 C CNN
-F 3 " https://product.tdk.com/info/en/catalog/datasheets/leadmlcc_halogenfree_fg_en.pdf?ref_disty=digikey" H 5550 4450 50  0001 C CNN
+F 3 " https://search.murata.co.jp/Ceramy/image/img/A01X/G101/ENG/RDE_X7R_250V-1kV_E.pdf" H 5550 4450 50  0001 C CNN
 F 4 "digikey" V 5550 4450 50  0001 C CNN "Vendor"
-F 5 "445-173474-1-ND" V 5550 4450 50  0001 C CNN "Vendor part#"
-F 6 "FG28C0G1H103JNT06" V 5550 4450 50  0001 C CNN "Manufacturer part#"
+F 5 "490-8814-ND" V 5550 4450 50  0001 C CNN "Vendor part#"
+F 6 "RDER71H104K0K1H03B" V 5550 4450 50  0001 C CNN "Manufacturer part#"
 	1    5550 4450
 	-1   0    0    1
